File: GingerLight.kicad_pcb (KiCad board)
At the start: 2 copper layers, 28 x 52.5 mm, 21 parts, among them J1 PWR, J2 LED, J3 PWM, Q1 CRSS052N08N

Commit message: Rev 1
Parts:
- C4: footprint Capacitor_SMD:C_0603_1608Metric_Pad1.08x0.95mm_HandSolder -> Capacitor_SMD:C_1206_3216Metric_Pad1.33x1.80mm_HandSolder
- moved R4 2.82 mm to (146.5, 120.0), turned to 0 degrees
- moved C5 1.89 mm to (143.9, 122.6)
- moved C4 0.87 mm to (151.4, 125.0)
- moved R501 0.09 mm to (154.6, 123.7)
Routing:
- net VBUS: track 100.5 -> 53.9 mm, vias 16 -> 12
- net LED+: track 46.1 -> 11.5 mm, vias 3 -> 0
- net LED-: track 9.65 -> 4.22 mm
- net Net-(Q1-S): track 19.2 -> 14.6 mm, vias 2 -> 0
- net GND: track 7.92 -> 3.40 mm, vias 53 -> 157
- net Net-(C301-Pad1): track 1.60 -> 3.31 mm
- added copper zone on F.Cu, net LED+
- added copper zone on F.Cu, net LED-
- added copper zone on F.Cu, net VBUS
Other:
- board text added: "+"
- board text added: "+12v"
- board text added: "36v 40w COB LED driver"
- board text added: "By Jackson M Hu (C) Feb 2024 Rev. 1"
- board text added: "GND"
- board text added: "LED+"
- board text added: "LED-"
- board text added: "PWM"

Commit message: Rev 1.1
Parts:
- added R101: 100k, Resistor_SMD:R_0603_1608Metric_Pad0.98x0.95mm_HandSolder, F.Cu at (146.9, 136.3)
- U1: value ~ -> CN5816
- moved R6 0.15 mm to (152.2, 130.9)
- moved R102 0.15 mm to (147.2, 131.2)
- renumbered R1 to R102
Connections:
- R102 pad 1: LED+ -> Net-(R101-Pad1)
Routing:
- net GND: track 3.40 -> 14.7 mm, vias 157 -> 177
- net LED+: track 11.5 -> 6.37 mm
- net Net-(R101-Pad1): track 0.00 -> 3.33 mm
- net LED-: track 4.22 -> 5.65 mm

Commit message: Rev 2
Parts:
- removed R101: 100k, Resistor_SMD:R_0603_1608Metric_Pad0.98x0.95mm_HandSolder
- C201, C202: value 10uF/50v -> 10uF/63v; footprint Capacitor_SMD:C_1206_3216Metric_Pad1.33x1.80mm_HandSolder -> Capacitor_SMD:C_1210_3225Metric_Pad1.33x2.70mm_HandSolder
- C301: value 100nF -> 120nF
- C302: value 47nF -> 1nF
- R1: renamed from R102; value 2740k -> 4220k
- R3: value 2.19k -> 5.8k
- R501, R502: value 0.1R/2w -> 0.09R/2w
- R6: value 0.1R/2w -> 0.15R/2w
- moved C201 1.34 mm to (156.5, 117.2)
- moved C202 0.37 mm to (156.5, 113.9)
- moved R1 0.16 mm to (147.1, 131.2)
Connections:
- R1 pad 1: Net-(R101-Pad1) -> LED+
Routing:
- net VBUS: track 53.9 -> 77.7 mm, vias 12 -> 19
- net LED+: track 6.37 -> 11.2 mm
- net GND: track 14.7 -> 10.4 mm, vias 177 -> 197
- net Net-(R101-Pad1): track 3.33 -> 0.00 mm
Other:
- board text added: "+20v"
- board text added: "By Jackson M Hu (C) March 2024 Rev. 2"
- board text removed: "+12v"
- board text removed: "By Jackson M Hu (C) Feb 2024 Rev. 1"
