File: GingerLight.kicad_sch (KiCad schematic)
At the start: 21 parts, among them J1 PWR, J2 LED, J3 PWM, Q1 CRSS052N08N

Commit message: Rev 1
Parts:
- C4: footprint Capacitor_SMD:C_0603_1608Metric_Pad1.08x0.95mm_HandSolder -> Capacitor_SMD:C_1206_3216Metric_Pad1.33x1.80mm_HandSolder
Other:
- note added: "Comment: - R1 value as per offical calculator suggest it should be 2861k"
Changed lines of the file:
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@@
     (stroke (width 0) (type default))
+  )
+  (text "Comment:\n\n- R1 value as per offical calculator suggest it should be 2861k"
+    (at 41.91 158.75 0)
+    (effects (font (size 1.27 1.27)) (justify left bottom))
   )
   (global_label "LED+" (shape input) (at 215.9 55.88 0) (fields_autoplaced)
@@
       (effects (font (size 1.27 1.27)) (justify left))
     )
-    (property "Footprint" "Capacitor_SMD:C_0603_1608Metric_Pad1.08x0.95mm_HandSolder" (at 77.1652 113.03 0)
-      (effects (font (size 1.27 1.27)) hide)
-    )
+    (property "Footprint" "Capacitor_SMD:C_1206_3216Metric_Pad1.33x1.80mm_HandSolder" (at 77.1652 113.03 0)
+      (effects (font (size 1.27 1.27)) hide)
+    )

Commit message: Rev 1.1
Parts:
- added R101: 100k, Resistor_SMD:R_0603_1608Metric_Pad0.98x0.95mm_HandSolder, symbol Device:R
- U1: value ~ -> CN5816
- renumbered R1 to R102
Connections:
- net LED+: now also R101.2; no longer R102.1
- new net: R101.1, R102.1
Changed lines of the file:
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@@
+    (stroke (width 0) (type default))
+  )
+  (wire (pts (xy 172.72 102.87) (xy 168.91 102.87))
     (stroke (width 0) (type default))
   )
@@
     (stroke (width 0) (type default))
   )
-  (wire (pts (xy 158.75 101.6) (xy 158.75 106.68))
-    (stroke (width 0) (type default))
-  )
   (wire (pts (xy 207.01 88.9) (xy 210.82 88.9))
     (stroke (width 0) (type default))
@@
     (stroke (width 0) (type default))
   )
+  (wire (pts (xy 161.29 102.87) (xy 158.75 102.87))
+    (stroke (width 0) (type default))
+  )
   (wire (pts (xy 142.24 69.85) (xy 142.24 73.66))
     (stroke (width 0) (type default))
@@
   )
   (wire (pts (xy 76.2 127) (xy 83.82 127))
+    (stroke (width 0) (type default))
+  )
+  (wire (pts (xy 158.75 102.87) (xy 158.75 106.68))
     (stroke (width 0) (type default))
   )
@@
     )
   )
-  (global_label "LED+" (shape input) (at 158.75 101.6 90) (fields_autoplaced)
+  (global_label "LED+" (shape input) (at 172.72 102.87 0) (fields_autoplaced)
     (effects (font (size 1.27 1.27)) (justify left))
-    (property "Intersheetrefs" "${INTERSHEET_REFS}" (at 158.75 93.5953 90)
+    (property "Intersheetrefs" "${INTERSHEET_REFS}" (at 180.7247 102.87 0)
       (effects (font (size 1.27 1.27)) (justify left) hide)
     )
@@
   )
   (symbol (lib_id "JackcoLib:CN5816") (at 120.65 88.9 0) (unit 1)
-    (in_bom yes) (on_board yes) (dnp no) (fields_autoplaced)
+    (in_bom yes) (on_board yes) (dnp no)
     (property "Reference" "U1" (at 122.8441 73.66 0)
       (effects (font (size 1.27 1.27)) (justify left))
     )
-    (property "Value" "~" (at 120.65 88.9 0)
+    (property "Value" "CN5816" (at 127 104.14 0)
       (effects (font (size 1.27 1.27)))
     )
@@
     )
   )
+  (symbol (lib_id "Device:R") (at 165.1 102.87 90) (unit 1)
+    (in_bom yes) (on_board yes) (dnp no) (fields_autoplaced)
+    (property "Reference" "R101" (at 165.1 96.52 90)
+      (effects (font (size 1.27 1.27)))
+    )
+    (property "Value" "100k" (at 165.1 99.06 90)
+      (effects (font (size 1.27 1.27)))
+    )
+    (property "Footprint" "Resistor_SMD:R_0603_1608Metric_Pad0.98x0.95mm_HandSolder" (at 165.1 104.648 90)
+      (effects (font (size 1.27 1.27)) hide)
+    )
+    (property "Datasheet" "~" (at 165.1 102.87 0)
+      (effects (font (size 1.27 1.27)) hide)
+    )
+    (pin "2")
+    (pin "1")
+    (instances
+      (project "GingerLight"
+        (path "/e422acb9-02d8-44d1-b8e8-54d13edc58dc"
+          (reference "R101") (unit 1)
+        )
+      )
+    )
+  )
   (symbol (lib_id "Device:C") (at 76.2 109.22 0) (unit 1)
     (in_bom yes) (on_board yes) (dnp no)
@@
   (symbol (lib_id "Device:R") (at 158.75 110.49 0) (unit 1)
     (in_bom yes) (on_board yes) (dnp no) (fields_autoplaced)
-    (property "Reference" "R1" (at 161.29 109.22 0)
+    (property "Reference" "R102" (at 161.29 109.22 0)
       (effects (font (size 1.27 1.27)) (justify left))
     )
@@
       (project "GingerLight"
         (path "/e422acb9-02d8-44d1-b8e8-54d13edc58dc"
-          (reference "R1") (unit 1)
-        )
-      )
+          (reference "R102") (unit 1)
+        )
+      )

Commit message: Rev 2
Parts:
- removed R101: 100k, Resistor_SMD:R_0603_1608Metric_Pad0.98x0.95mm_HandSolder, symbol Device:R
- C201, C202: value 10uF/50v -> 10uF/63v; footprint Capacitor_SMD:C_1206_3216Metric_Pad1.33x1.80mm_HandSolder -> Capacitor_SMD:C_1210_3225Metric_Pad1.33x2.70mm_HandSolder
- C301: value 100nF -> 120nF
- C302: value 47nF -> 1nF
- R1: renamed from R102; value 2740k -> 4220k
- R3: value 2.19k -> 5.8k
- R501, R502: value 0.1R/2w -> 0.09R/2w
- R6: value 0.1R/2w -> 0.15R/2w
Connections:
- net LED+: now also R1.1
Other:
- note added: "Comment: - R1 (R101+R102) value as per offical calculator suggest it should be 4420k, but datasheet says it's 4260k - Voltage threshold is NOT just 36v, it's 56v (20+36v)!!! - R5 (R501+R502) value needs to be 0.045ohm, but probably 0.05ohm is fine too - If the LED become smoky, change R6 (Rcs) to 0.15ohm or 0.2ohm."
- note removed: "Comment: - R1 value as per offical calculator suggest it should be 2861k"
